File: naa_g/naa_g.sch (KiCad schematic (older format))
At the start: 29 parts, among them X1 Check_point, X2 Check_point, X3 Check_point, X4 LOGO_NIKITOS_19х7

Commit message: обновлена PDF
Parts:
- C3: value Конденсатор_16В_0.1_мкФ+-10проц. -> Конденсатор_16В_47_пФ+-10проц.
- X1, X2, X3: INFO (none) -> PCB_element
Changed lines of the file:
@@
 EESchema Schematic File Version 4
+LIBS:naa_g-cache
 EELAYER 30 0
 EELAYER END
@@
 F 2 "N_X:Пробник" H 5600 3000 50  0001 C CNN
 F 3 "" H 5600 3000 50  0001 C CNN
+F 4 "PCB_element" H 5600 3000 50  0001 C CNN "INFO"
 	1    5600 3000
 	1    0    0    -1
@@
 P 3800 6350
 F 0 "C3" V 3850 6200 60  0000 C CNN
-F 1 "Конденсатор_16В_0.1_мкФ+-10проц." H 3750 6100 60  0001 C CNN
+F 1 "Конденсатор_16В_47_пФ+-10проц." H 3750 6100 60  0001 C CNN
 F 2 "MOTOR_RLC:Конденсатор_SMD_К10-83(0603)" H 3700 6200 60  0001 C CNN
 F 3 "${MOTOR_2020_LIB}\\documentation\\IMPORT\\murata_smd_ceramic_cap.pdf" H 3800 6350 60  0001 C CNN
@@
 F 2 "N_X:Пробник" H 3500 3600 50  0001 C CNN
 F 3 "" H 3500 3600 50  0001 C CNN
+F 4 "PCB_element" H 3500 3600 50  0001 C CNN "INFO"
 	1    3500 3600
 	0    -1   -1   0
@@
 F 2 "N_X:Пробник" H 3500 2100 50  0001 C CNN
 F 3 "" H 3500 2100 50  0001 C CNN
+F 4 "PCB_element" H 3500 2100 50  0001 C CNN "INFO"
 	1    3500 2100
 	0    -1   -1   0
